File: PCB/IR_LED.sch (KiCad schematic (older format))
At the start: 7 parts

Commit message: DXFを追加、部品配置を開始
Parts:
- D4, D5: renamed from D?; footprint (none) -> LED_THT:LED_D5.0mm_Horizontal_O6.35mm_Z9.0mm
- Q3: renamed from Q?; footprint (none) -> Package_TO_SOT_THT:SIPAK_Vertical
- R10, R11, R9: renamed from R?; footprint (none) -> Resistor_THT:R_Axial_DIN0207_L6.3mm_D2.5mm_P7.62mm_Horizontal
- U2: renamed from U?; footprint (none) -> Package_DIP:DIP-8_W7.62mm_Socket
Changed lines of the file:
@@
 $EndDescr
 $Comp
-L Cheese_Burger_Library:NJM2742D U?
+L Cheese_Burger_Library:NJM2742D U2
 U 2 1 5EA2B92A
 P 2150 1700
-AR Path="/5EA07A67/5EA2B92A" Ref="U?"  Part="1"
-AR Path="/5EA2C744/5EA2B92A" Ref="U?"  Part="2"
-F 0 "U?" H 2150 1900 50  0000 L CNN
+AR Path="/5EA07A67/5EA2B92A" Ref="U2"  Part="2"
+AR Path="/5EA2C744/5EA2B92A" Ref="U2"  Part="1"
+F 0 "U2" H 2150 1900 50  0000 L CNN
 F 1 "NJM2742D" H 2150 1500 50  0000 L CNN
-F 2 "" H 2150 1700 50  0001 C CNN
+F 2 "Package_DIP:DIP-8_W7.62mm_Socket" H 2150 1700 50  0001 C CNN
 F 3 "" H 2150 1700 50  0001 C CNN
 	2    2150 1700
@@
 $EndComp
 $Comp
-L power:GND #PWR?
+L power:GND #PWR0115
 U 1 1 5EA2B9BF
 P 2050 2100
-AR Path="/5EA07A67/5EA2B9BF" Ref="#PWR?"  Part="1"
-AR Path="/5EA2C744/5EA2B9BF" Ref="#PWR?"  Part="1"
-F 0 "#PWR?" H 2050 1850 50  0001 C CNN
+AR Path="/5EA07A67/5EA2B9BF" Ref="#PWR0115"  Part="1"
+AR Path="/5EA2C744/5EA2B9BF" Ref="#PWR0108"  Part="1"
+F 0 "#PWR0115" H 2050 1850 50  0001 C CNN
 F 1 "GND" H 2055 1927 50  0000 C CNN
 F 2 "" H 2050 2100 50  0001 C CNN
@@
 $EndComp
 $Comp
-L Device:R R?
+L Device:R R10
 U 1 1 5EA2BA2E
 P 2600 1700
-AR Path="/5EA07A67/5EA2BA2E" Ref="R?"  Part="1"
-AR Path="/5EA2C744/5EA2BA2E" Ref="R?"  Part="1"
-F 0 "R?" V 2393 1700 50  0000 C CNN
+AR Path="/5EA07A67/5EA2BA2E" Ref="R10"  Part="1"
+AR Path="/5EA2C744/5EA2BA2E" Ref="R7"  Part="1"
+F 0 "R10" V 2393 1700 50  0000 C CNN
 F 1 "10" V 2484 1700 50  0000 C CNN
-F 2 "" V 2530 1700 50  0001 C CNN
+F 2 "Resistor_THT:R_Axial_DIN0207_L6.3mm_D2.5mm_P7.62mm_Horizontal" V 2530 1700 50  0001 C CNN
 F 3 "~" H 2600 1700 50  0001 C CNN
 	1    2600 1700
@@
 $EndComp
 $Comp
-L Device:R R?
+L Device:R R9
 U 1 1 5EA2BA71
 P 1400 1750
-AR Path="/5EA07A67/5EA2BA71" Ref="R?"  Part="1"
-AR Path="/5EA2C744/5EA2BA71" Ref="R?"  Part="1"
-F 0 "R?" H 1330 1704 50  0000 R CNN
+AR Path="/5EA07A67/5EA2BA71" Ref="R9"  Part="1"
+AR Path="/5EA2C744/5EA2BA71" Ref="R6"  Part="1"
+F 0 "R9" H 1330 1704 50  0000 R CNN
 F 1 "10k" H 1330 1795 50  0000 R CNN
-F 2 "" V 1330 1750 50  0001 C CNN
+F 2 "Resistor_THT:R_Axial_DIN0207_L6.3mm_D2.5mm_P7.62mm_Horizontal" V 1330 1750 50  0001 C CNN
 F 3 "~" H 1400 1750 50  0001 C CNN
 	1    1400 1750
@@
 $EndComp
 $Comp
-L power:GND #PWR?
+L power:GND #PWR0116
 U 1 1 5EA2BADF
 P 1400 1900
-AR Path="/5EA07A67/5EA2BADF" Ref="#PWR?"  Part="1"
-AR Path="/5EA2C744/5EA2BADF" Ref="#PWR?"  Part="1"
-F 0 "#PWR?" H 1400 1650 50  0001 C CNN
+AR Path="/5EA07A67/5EA2BADF" Ref="#PWR0116"  Part="1"
+AR Path="/5EA2C744/5EA2BADF" Ref="#PWR0109"  Part="1"
+F 0 "#PWR0116" H 1400 1650 50  0001 C CNN
 F 1 "GND" H 1405 1727 50  0000 C CNN
 F 2 "" H 1400 1900 50  0001 C CNN
@@
 	1750 1800 1750 2350
 $Comp
-L Device:Q_NMOS_GDS Q?
+L Device:Q_NMOS_GDS Q3
 U 1 1 5EA2BC4E
 P 2950 1700
-AR Path="/5EA07A67/5EA2BC4E" Ref="Q?"  Part="1"
-AR Path="/5EA2C744/5EA2BC4E" Ref="Q?"  Part="1"
-F 0 "Q?" H 3155 1746 50  0000 L CNN
+AR Path="/5EA07A67/5EA2BC4E" Ref="Q3"  Part="1"
+AR Path="/5EA2C744/5EA2BC4E" Ref="Q2"  Part="1"
+F 0 "Q3" H 3155 1746 50  0000 L CNN
 F 1 "2SK2796" H 3155 1655 50  0000 L CNN
-F 2 "" H 3150 1800 50  0001 C CNN
+F 2 "Package_TO_SOT_THT:SIPAK_Vertical" H 3150 1800 50  0001 C CNN
 F 3 "~" H 2950 1700 50  0001 C CNN
 	1    2950 1700
@@
 	1750 2350 3050 2350
 $Comp
-L Device:R R?
+L Device:R R11
 U 1 1 5EA2BCE2
 P 3050 2500
-AR Path="/5EA07A67/5EA2BCE2" Ref="R?"  Part="1"
-AR Path="/5EA2C744/5EA2BCE2" Ref="R?"  Part="1"
-F 0 "R?" H 2980 2454 50  0000 R CNN
+AR Path="/5EA07A67/5EA2BCE2" Ref="R11"  Part="1"
+AR Path="/5EA2C744/5EA2BCE2" Ref="R8"  Part="1"
+F 0 "R11" H 2980 2454 50  0000 R CNN
 F 1 "33 1/2W 1%" H 2980 2545 50  0000 R CNN
-F 2 "" V 2980 2500 50  0001 C CNN
+F 2 "Resistor_THT:R_Axial_DIN0207_L6.3mm_D2.5mm_P7.62mm_Horizontal" V 2980 2500 50  0001 C CNN
 F 3 "~" H 3050 2500 50  0001 C CNN
 	1    3050 2500
@@
 Connection ~ 3050 2350
 $Comp
-L power:GND #PWR?
+L power:GND #PWR0117
 U 1 1 5EA2BD4F
 P 3050 2650
-AR Path="/5EA07A67/5EA2BD4F" Ref="#PWR?"  Part="1"
-AR Path="/5EA2C744/5EA2BD4F" Ref="#PWR?"  Part="1"
-F 0 "#PWR?" H 3050 2400 50  0001 C CNN
+AR Path="/5EA07A67/5EA2BD4F" Ref="#PWR0117"  Part="1"
+AR Path="/5EA2C744/5EA2BD4F" Ref="#PWR0110"  Part="1"
+F 0 "#PWR0117" H 3050 2400 50  0001 C CNN
 F 1 "GND" H 3055 2477 50  0000 C CNN
 F 2 "" H 3050 2650 50  0001 C CNN
@@
 	1400 1600 1850 1600
 $Comp
-L Device:LED_ALT D?
+L Device:LED_ALT D5
 U 1 1 5EA2BE25
 P 3050 1250
-AR Path="/5EA07A67/5EA2BE25" Ref="D?"  Part="1"
-AR Path="/5EA2C744/5EA2BE25" Ref="D?"  Part="1"
-F 0 "D?" V 3088 1132 50  0000 R CNN
+AR Path="/5EA07A67/5EA2BE25" Ref="D5"  Part="1"
+AR Path="/5EA2C744/5EA2BE25" Ref="D3"  Part="1"
+F 0 "D5" V 3088 1132 50  0000 R CNN
 F 1 "LED_ALT" V 2997 1132 50  0000 R CNN
-F 2 "" H 3050 1250 50  0001 C CNN
+F 2 "LED_THT:LED_D5.0mm_Horizontal_O6.35mm_Z9.0mm" H 3050 1250 50  0001 C CNN
 F 3 "~" H 3050 1250 50  0001 C CNN
 	1    3050 1250
@@
 $EndComp
 $Comp
-L Device:LED_ALT D?
+L Device:LED_ALT D4
 U 1 1 5EA2BE84
 P 3050 950
-AR Path="/5EA07A67/5EA2BE84" Ref="D?"  Part="1"
-AR Path="/5EA2C744/5EA2BE84" Ref="D?"  Part="1"
-F 0 "D?" V 3088 832 50  0000 R CNN
+AR Path="/5EA07A67/5EA2BE84" Ref="D4"  Part="1"
+AR Path="/5EA2C744/5EA2BE84" Ref="D2"  Part="1"
+F 0 "D4" V 3088 832 50  0000 R CNN
 F 1 "LED_ALT" V 2997 832 50  0000 R CNN
-F 2 "" H 3050 950 50  0001 C CNN
+F 2 "LED_THT:LED_D5.0mm_Horizontal_O6.35mm_Z9.0mm" H 3050 950 50  0001 C CNN
 F 3 "~" H 3050 950 50  0001 C CNN
 	1    3050 950
@@
 	3050 1500 3050 1400
 $Comp
-L power:+BATT #PWR?
+L power:+BATT #PWR0118
 U 1 1 5EA2BEEB
 P 3050 800
-AR Path="/5EA07A67/5EA2BEEB" Ref="#PWR?"  Part="1"
-AR Path="/5EA2C744/5EA2BEEB" Ref="#PWR?"  Part="1"
-F 0 "#PWR?" H 3050 650 50  0001 C CNN
+AR Path="/5EA07A67/5EA2BEEB" Ref="#PWR0118"  Part="1"
+AR Path="/5EA2C744/5EA2BEEB" Ref="#PWR0111"  Part="1"
+F 0 "#PWR0118" H 3050 650 50  0001 C CNN
 F 1 "+BATT" H 3065 973 50  0000 C CNN
 F 2 "" H 3050 800 50  0001 C CNN
@@
 	2050 1450 2050 1250
 $Comp
-L power:+BATT #PWR?
+L power:+BATT #PWR0119
 U 1 1 5EA2B986
 P 2050 1250
-AR Path="/5EA07A67/5EA2B986" Ref="#PWR?"  Part="1"
-AR Path="/5EA2C744/5EA2B986" Ref="#PWR?"  Part="1"
-F 0 "#PWR?" H 2050 1100 50  0001 C CNN
+AR Path="/5EA07A67/5EA2B986" Ref="#PWR0119"  Part="1"
+AR Path="/5EA2C744/5EA2B986" Ref="#PWR0112"  Part="1"
+F 0 "#PWR0119" H 2050 1100 50  0001 C CNN
 F 1 "+BATT" H 2065 1423 50  0000 C CNN
 F 2 "" H 2050 1250 50  0001 C CNN
@@
 $EndComp
 $Comp
-L power:GND #PWR?
+L power:GND #PWR0120
 U 1 1 5EA2C0C1
 P 1400 1050
-AR Path="/5EA07A67/5EA2C0C1" Ref="#PWR?"  Part="1"
-AR Path="/5EA2C744/5EA2C0C1" Ref="#PWR?"  Part="1"
-F 0 "#PWR?" H 1400 800 50  0001 C CNN
+AR Path="/5EA07A67/5EA2C0C1" Ref="#PWR0120"  Part="1"
+AR Path="/5EA2C744/5EA2C0C1" Ref="#PWR0113"  Part="1"
+F 0 "#PWR0120" H 1400 800 50  0001 C CNN
 F 1 "GND" H 1405 877 50  0000 C CNN
 F 2 "" H 1400 1050 50  0001 C CNN
@@
 $EndComp
 $Comp
-L power:+BATT #PWR?
+L power:+BATT #PWR0121
 U 1 1 5EA2C106
 P 1400 850
-AR Path="/5EA07A67/5EA2C106" Ref="#PWR?"  Part="1"
-AR Path="/5EA2C744/5EA2C106" Ref="#PWR?"  Part="1"
-F 0 "#PWR?" H 1400 700 50  0001 C CNN
+AR Path="/5EA07A67/5EA2C106" Ref="#PWR0121"  Part="1"
+AR Path="/5EA2C744/5EA2C106" Ref="#PWR0114"  Part="1"
+F 0 "#PWR0121" H 1400 700 50  0001 C CNN
 F 1 "+BATT" H 1415 1023 50  0000 C CNN
 F 2 "" H 1400 850 50  0001 C CNN
