File: PCB/IR_Sensor.sch (KiCad schematic (older format))
At the start: 6 parts

Commit message: DXFを追加、部品配置を開始
Parts:
- C3, C4: renamed from C?; footprint (none) -> Capacitor_THT:C_Disc_D5.0mm_W2.5mm_P5.00mm
- D6: renamed from D?; footprint (none) -> LED_THT:LED_D5.0mm_Horizontal_O3.81mm_Z3.0mm
- R12, R13: renamed from R?; footprint (none) -> Resistor_THT:R_Axial_DIN0207_L6.3mm_D2.5mm_P7.62mm_Horizontal
- U3: renamed from U?; footprint (none) -> Package_DIP:DIP-8_W7.62mm_Socket
Changed lines of the file:
@@
 $EndDescr
 $Comp
-L Cheese_Burger_Library:NJU7072D U?
+L Cheese_Burger_Library:NJU7072D U3
 U 2 1 5EA2CADB
 P 2450 2400
-AR Path="/5EA2C81D/5EA2CADB" Ref="U?"  Part="1"
-AR Path="/5EA2D9F0/5EA2CADB" Ref="U?"  Part="2"
-AR Path="/5EA2D9F3/5EA2CADB" Ref="U?"  Part="1"
-AR Path="/5EA2D9F6/5EA2CADB" Ref="U?"  Part="2"
-F 0 "U?" H 2450 2600 50  0000 L CNN
+AR Path="/5EA2C81D/5EA2CADB" Ref="U3"  Part="1"
+AR Path="/5EA2D9F0/5EA2CADB" Ref="U3"  Part="2"
+AR Path="/5EA2D9F3/5EA2CADB" Ref="U4"  Part="1"
+AR Path="/5EA2D9F6/5EA2CADB" Ref="U4"  Part="2"
+F 0 "U4" H 2450 2600 50  0000 L CNN
 F 1 "NJU7072D" H 2450 2200 50  0000 L CNN
-F 2 "" H 2450 2400 50  0001 C CNN
+F 2 "Package_DIP:DIP-8_W7.62mm_Socket" H 2450 2400 50  0001 C CNN
 F 3 "" H 2450 2400 50  0001 C CNN
 	2    2450 2400
@@
 $EndComp
 $Comp
-L power:+3.3VA #PWR?
+L power:+3.3VA #PWR0122
 U 1 1 5EA2CB66
 P 2350 2150
-AR Path="/5EA2C81D/5EA2CB66" Ref="#PWR?"  Part="1"
-AR Path="/5EA2D9F0/5EA2CB66" Ref="#PWR?"  Part="1"
-AR Path="/5EA2D9F3/5EA2CB66" Ref="#PWR?"  Part="1"
-AR Path="/5EA2D9F6/5EA2CB66" Ref="#PWR?"  Part="1"
-F 0 "#PWR?" H 2350 2000 50  0001 C CNN
+AR Path="/5EA2C81D/5EA2CB66" Ref="#PWR0122"  Part="1"
+AR Path="/5EA2D9F0/5EA2CB66" Ref="#PWR0128"  Part="1"
+AR Path="/5EA2D9F3/5EA2CB66" Ref="#PWR0134"  Part="1"
+AR Path="/5EA2D9F6/5EA2CB66" Ref="#PWR0140"  Part="1"
+F 0 "#PWR0140" H 2350 2000 50  0001 C CNN
 F 1 "+3.3VA" H 2365 2323 50  0000 C CNN
 F 2 "" H 2350 2150 50  0001 C CNN
@@
 $EndComp
 $Comp
-L Device:R R?
+L Device:R R13
 U 1 1 5EA2CB98
 P 2350 1850
-AR Path="/5EA2C81D/5EA2CB98" Ref="R?"  Part="1"
-AR Path="/5EA2D9F0/5EA2CB98" Ref="R?"  Part="1"
-AR Path="/5EA2D9F3/5EA2CB98" Ref="R?"  Part="1"
-AR Path="/5EA2D9F6/5EA2CB98" Ref="R?"  Part="1"
-F 0 "R?" V 2143 1850 50  0000 C CNN
+AR Path="/5EA2C81D/5EA2CB98" Ref="R13"  Part="1"
+AR Path="/5EA2D9F0/5EA2CB98" Ref="R15"  Part="1"
+AR Path="/5EA2D9F3/5EA2CB98" Ref="R17"  Part="1"
+AR Path="/5EA2D9F6/5EA2CB98" Ref="R19"  Part="1"
+F 0 "R19" V 2143 1850 50  0000 C CNN
 F 1 "220k" V 2234 1850 50  0000 C CNN
-F 2 "" V 2280 1850 50  0001 C CNN
+F 2 "Resistor_THT:R_Axial_DIN0207_L6.3mm_D2.5mm_P7.62mm_Horizontal" V 2280 1850 50  0001 C CNN
 F 3 "~" H 2350 1850 50  0001 C CNN
 	1    2350 1850
@@
 $EndComp
 $Comp
-L Device:C C?
+L Device:C C4
 U 1 1 5EA2CC2D
 P 2350 1500
-AR Path="/5EA2C81D/5EA2CC2D" Ref="C?"  Part="1"
-AR Path="/5EA2D9F0/5EA2CC2D" Ref="C?"  Part="1"
-AR Path="/5EA2D9F3/5EA2CC2D" Ref="C?"  Part="1"
-AR Path="/5EA2D9F6/5EA2CC2D" Ref="C?"  Part="1"
-F 0 "C?" V 2098 1500 50  0000 C CNN
+AR Path="/5EA2C81D/5EA2CC2D" Ref="C4"  Part="1"
+AR Path="/5EA2D9F0/5EA2CC2D" Ref="C6"  Part="1"
+AR Path="/5EA2D9F3/5EA2CC2D" Ref="C8"  Part="1"
+AR Path="/5EA2D9F6/5EA2CC2D" Ref="C10"  Part="1"
+F 0 "C10" V 2098 1500 50  0000 C CNN
 F 1 "22p" V 2189 1500 50  0000 C CNN
-F 2 "" H 2388 1350 50  0001 C CNN
+F 2 "Capacitor_THT:C_Disc_D5.0mm_W2.5mm_P5.00mm" H 2388 1350 50  0001 C CNN
 F 3 "~" H 2350 1500 50  0001 C CNN
 	1    2350 1500
@@
 1.65V
 $Comp
-L Device:C C?
+L Device:C C3
 U 1 1 5EA2CFD2
 P 1550 2500
-AR Path="/5EA2C81D/5EA2CFD2" Ref="C?"  Part="1"
-AR Path="/5EA2D9F0/5EA2CFD2" Ref="C?"  Part="1"
-AR Path="/5EA2D9F3/5EA2CFD2" Ref="C?"  Part="1"
-AR Path="/5EA2D9F6/5EA2CFD2" Ref="C?"  Part="1"
-F 0 "C?" V 1298 2500 50  0000 C CNN
+AR Path="/5EA2C81D/5EA2CFD2" Ref="C3"  Part="1"
+AR Path="/5EA2D9F0/5EA2CFD2" Ref="C5"  Part="1"
+AR Path="/5EA2D9F3/5EA2CFD2" Ref="C7"  Part="1"
+AR Path="/5EA2D9F6/5EA2CFD2" Ref="C9"  Part="1"
+F 0 "C9" V 1298 2500 50  0000 C CNN
 F 1 "22p" V 1389 2500 50  0000 C CNN
-F 2 "" H 1588 2350 50  0001 C CNN
+F 2 "Capacitor_THT:C_Disc_D5.0mm_W2.5mm_P5.00mm" H 1588 2350 50  0001 C CNN
 F 3 "~" H 1550 2500 50  0001 C CNN
 	1    1550 2500
@@
 $EndComp
 $Comp
-L Device:R R?
+L Device:R R12
 U 1 1 5EA2D012
 P 1400 2800
-AR Path="/5EA2C81D/5EA2D012" Ref="R?"  Part="1"
-AR Path="/5EA2D9F0/5EA2D012" Ref="R?"  Part="1"
-AR Path="/5EA2D9F3/5EA2D012" Ref="R?"  Part="1"
-AR Path="/5EA2D9F6/5EA2D012" Ref="R?"  Part="1"
-F 0 "R?" H 1330 2754 50  0000 R CNN
+AR Path="/5EA2C81D/5EA2D012" Ref="R12"  Part="1"
+AR Path="/5EA2D9F0/5EA2D012" Ref="R14"  Part="1"
+AR Path="/5EA2D9F3/5EA2D012" Ref="R16"  Part="1"
+AR Path="/5EA2D9F6/5EA2D012" Ref="R18"  Part="1"
+F 0 "R18" H 1330 2754 50  0000 R CNN
 F 1 "220k" H 1330 2845 50  0000 R CNN
-F 2 "" V 1330 2800 50  0001 C CNN
+F 2 "Resistor_THT:R_Axial_DIN0207_L6.3mm_D2.5mm_P7.62mm_Horizontal" V 1330 2800 50  0001 C CNN
 F 3 "~" H 1400 2800 50  0001 C CNN
 	1    1400 2800
@@
 Connection ~ 1800 2500
 $Comp
-L power:GND #PWR?
+L power:GND #PWR0123
 U 1 1 5EA2D1CF
 P 1400 2950
-AR Path="/5EA2C81D/5EA2D1CF" Ref="#PWR?"  Part="1"
-AR Path="/5EA2D9F0/5EA2D1CF" Ref="#PWR?"  Part="1"
-AR Path="/5EA2D9F3/5EA2D1CF" Ref="#PWR?"  Part="1"
-AR Path="/5EA2D9F6/5EA2D1CF" Ref="#PWR?"  Part="1"
-F 0 "#PWR?" H 1400 2700 50  0001 C CNN
+AR Path="/5EA2C81D/5EA2D1CF" Ref="#PWR0123"  Part="1"
+AR Path="/5EA2D9F0/5EA2D1CF" Ref="#PWR0129"  Part="1"
+AR Path="/5EA2D9F3/5EA2D1CF" Ref="#PWR0135"  Part="1"
+AR Path="/5EA2D9F6/5EA2D1CF" Ref="#PWR0141"  Part="1"
+F 0 "#PWR0141" H 1400 2700 50  0001 C CNN
 F 1 "GND" H 1405 2777 50  0000 C CNN
 F 2 "" H 1400 2950 50  0001 C CNN
@@
 $EndComp
 $Comp
-L power:+3.3VA #PWR?
+L power:+3.3VA #PWR0124
 U 1 1 5EA2D1EB
 P 1400 1850
-AR Path="/5EA2C81D/5EA2D1EB" Ref="#PWR?"  Part="1"
-AR Path="/5EA2D9F0/5EA2D1EB" Ref="#PWR?"  Part="1"
-AR Path="/5EA2D9F3/5EA2D1EB" Ref="#PWR?"  Part="1"
-AR Path="/5EA2D9F6/5EA2D1EB" Ref="#PWR?"  Part="1"
-F 0 "#PWR?" H 1400 1700 50  0001 C CNN
+AR Path="/5EA2C81D/5EA2D1EB" Ref="#PWR0124"  Part="1"
+AR Path="/5EA2D9F0/5EA2D1EB" Ref="#PWR0130"  Part="1"
+AR Path="/5EA2D9F3/5EA2D1EB" Ref="#PWR0136"  Part="1"
+AR Path="/5EA2D9F6/5EA2D1EB" Ref="#PWR0142"  Part="1"
+F 0 "#PWR0142" H 1400 1700 50  0001 C CNN
 F 1 "+3.3VA" H 1415 2023 50  0000 C CNN
 F 2 "" H 1400 1850 50  0001 C CNN
@@
 $EndComp
 $Comp
-L Device:D_Photo_ALT D?
+L Device:D_Photo_ALT D6
 U 1 1 5EA2D233
 P 1400 2150
-AR Path="/5EA2C81D/5EA2D233" Ref="D?"  Part="1"
-AR Path="/5EA2D9F0/5EA2D233" Ref="D?"  Part="1"
-AR Path="/5EA2D9F3/5EA2D233" Ref="D?"  Part="1"
-AR Path="/5EA2D9F6/5EA2D233" Ref="D?"  Part="1"
-F 0 "D?" V 1300 1600 50  0000 L CNN
+AR Path="/5EA2C81D/5EA2D233" Ref="D6"  Part="1"
+AR Path="/5EA2D9F0/5EA2D233" Ref="D7"  Part="1"
+AR Path="/5EA2D9F3/5EA2D233" Ref="D8"  Part="1"
+AR Path="/5EA2D9F6/5EA2D233" Ref="D9"  Part="1"
+F 0 "D9" V 1300 1600 50  0000 L CNN
 F 1 "D_Photo_ALT" V 1400 1600 50  0000 L CNN
-F 2 "" H 1350 2150 50  0001 C CNN
+F 2 "LED_THT:LED_D5.0mm_Horizontal_O3.81mm_Z3.0mm" H 1350 2150 50  0001 C CNN
 F 3 "~" H 1350 2150 50  0001 C CNN
 	1    1400 2150
@@
 	1400 1950 1400 1850
 $Comp
-L power:GND #PWR?
+L power:GND #PWR0125
 U 1 1 5EA2D4B8
 P 2350 2950
-AR Path="/5EA2C81D/5EA2D4B8" Ref="#PWR?"  Part="1"
-AR Path="/5EA2D9F0/5EA2D4B8" Ref="#PWR?"  Part="1"
-AR Path="/5EA2D9F3/5EA2D4B8" Ref="#PWR?"  Part="1"
-AR Path="/5EA2D9F6/5EA2D4B8" Ref="#PWR?"  Part="1"
-F 0 "#PWR?" H 2350 2700 50  0001 C CNN
+AR Path="/5EA2C81D/5EA2D4B8" Ref="#PWR0125"  Part="1"
+AR Path="/5EA2D9F0/5EA2D4B8" Ref="#PWR0131"  Part="1"
+AR Path="/5EA2D9F3/5EA2D4B8" Ref="#PWR0137"  Part="1"
+AR Path="/5EA2D9F6/5EA2D4B8" Ref="#PWR0143"  Part="1"
+F 0 "#PWR0143" H 2350 2700 50  0001 C CNN
 F 1 "GND" H 2355 2777 50  0000 C CNN
 F 2 "" H 2350 2950 50  0001 C CNN
@@
 	2350 2950 2350 2650
 $Comp
-L power:GND #PWR?
+L power:GND #PWR0126
 U 1 1 5EA2D5E7
 P 3400 2000
-AR Path="/5EA2C81D/5EA2D5E7" Ref="#PWR?"  Part="1"
-AR Path="/5EA2D9F0/5EA2D5E7" Ref="#PWR?"  Part="1"
-AR Path="/5EA2D9F3/5EA2D5E7" Ref="#PWR?"  Part="1"
-AR Path="/5EA2D9F6/5EA2D5E7" Ref="#PWR?"  Part="1"
-F 0 "#PWR?" H 3400 1750 50  0001 C CNN
+AR Path="/5EA2C81D/5EA2D5E7" Ref="#PWR0126"  Part="1"
+AR Path="/5EA2D9F0/5EA2D5E7" Ref="#PWR0132"  Part="1"
+AR Path="/5EA2D9F3/5EA2D5E7" Ref="#PWR0138"  Part="1"
+AR Path="/5EA2D9F6/5EA2D5E7" Ref="#PWR0144"  Part="1"
+F 0 "#PWR0144" H 3400 1750 50  0001 C CNN
 F 1 "GND" H 3405 1827 50  0000 C CNN
 F 2 "" H 3400 2000 50  0001 C CNN
@@
 $EndComp
 $Comp
-L power:+3.3VA #PWR?
+L power:+3.3VA #PWR0127
 U 1 1 5EA2D5FE
 P 3400 1750
-AR Path="/5EA2C81D/5EA2D5FE" Ref="#PWR?"  Part="1"
-AR Path="/5EA2D9F0/5EA2D5FE" Ref="#PWR?"  Part="1"
-AR Path="/5EA2D9F3/5EA2D5FE" Ref="#PWR?"  Part="1"
-AR Path="/5EA2D9F6/5EA2D5FE" Ref="#PWR?"  Part="1"
-F 0 "#PWR?" H 3400 1600 50  0001 C CNN
+AR Path="/5EA2C81D/5EA2D5FE" Ref="#PWR0127"  Part="1"
+AR Path="/5EA2D9F0/5EA2D5FE" Ref="#PWR0133"  Part="1"
+AR Path="/5EA2D9F3/5EA2D5FE" Ref="#PWR0139"  Part="1"
+AR Path="/5EA2D9F6/5EA2D5FE" Ref="#PWR0145"  Part="1"
+F 0 "#PWR0145" H 3400 1600 50  0001 C CNN
 F 1 "+3.3VA" H 3415 1923 50  0000 C CNN
 F 2 "" H 3400 1750 50  0001 C CNN
