File: PCB/Power.sch (KiCad schematic (older format))
At the start: 14 parts

Commit message: DXFを追加、部品配置を開始
Parts:
- C1, C2: renamed from C?; footprint (none) -> Capacitor_THT:C_Disc_D5.0mm_W2.5mm_P5.00mm
- D1: renamed from D?; footprint (none) -> LED_THT:LED_D5.0mm
- F1: renamed from F?; value RXEF160 -> MF-RX160; footprint (none) -> Cheese_Burger_Library:RF-RX160
- J2: renamed from J?; footprint (none) -> Connector_JST:JST_XH_B02B-XH-A_1x02_P2.50mm_Vertical
- L1: renamed from L?; footprint (none) -> Inductor_THT:L_Axial_L7.0mm_D3.3mm_P10.16mm_Horizontal_Fastron_MICC
- Q1: renamed from Q?; footprint (none) -> Package_TO_SOT_THT:SIPAK_Vertical
- R1, R2, R3, R4, R5: renamed from R?; footprint (none) -> Resistor_THT:R_Axial_DIN0207_L6.3mm_D2.5mm_P7.62mm_Horizontal
- SW1: renamed from SW?; footprint (none) -> Connector_PinHeader_2.54mm:PinHeader_1x03_P2.54mm_Vertical
- gave numbers to parts that had none: 1
Connections:
- wire segments 39 -> 41
Changed lines of the file:
@@
 $EndDescr
 $Comp
-L Connector_Generic:Conn_01x02 J?
+L Connector_Generic:Conn_01x02 J2
 U 1 1 5EA0036D
 P 1950 1600
-F 0 "J?" H 1870 1817 50  0000 C CNN
+F 0 "J2" H 1870 1817 50  0000 C CNN
 F 1 "JST_XA_1x2" H 1870 1726 50  0000 C CNN
-F 2 "" H 1950 1600 50  0001 C CNN
+F 2 "Connector_JST:JST_XH_B02B-XH-A_1x02_P2.50mm_Vertical" H 1950 1600 50  0001 C CNN
 F 3 "~" H 1950 1600 50  0001 C CNN
 	1    1950 1600
@@
 $EndComp
 $Comp
-L Device:Polyfuse F?
+L Device:Polyfuse F1
 U 1 1 5EA00419
 P 2550 1600
-F 0 "F?" V 2325 1600 50  0000 C CNN
-F 1 "RXEF160" V 2416 1600 50  0000 C CNN
-F 2 "" H 2600 1400 50  0001 L CNN
+F 0 "F1" V 2325 1600 50  0000 C CNN
+F 1 "MF-RX160" V 2416 1600 50  0000 C CNN
+F 2 "Cheese_Burger_Library:RF-RX160" H 2600 1400 50  0001 L CNN
 F 3 "~" H 2550 1600 50  0001 C CNN
 	1    2550 1600
@@
 11.1V
 $Comp
-L Device:Q_NMOS_GDS Q?
+L Device:Q_NMOS_GDS Q1
 U 1 1 5EA0084F
 P 3100 1700
-F 0 "Q?" V 3443 1700 50  0000 C CNN
+F 0 "Q1" V 3443 1700 50  0000 C CNN
 F 1 "2SK4017" V 3352 1700 50  0000 C CNN
-F 2 "" H 3300 1800 50  0001 C CNN
+F 2 "Package_TO_SOT_THT:SIPAK_Vertical" H 3300 1800 50  0001 C CNN
 F 3 "~" H 3100 1700 50  0001 C CNN
 	1    3100 1700
@@
 	2150 1700 2250 1700
 $Comp
-L power:GND #PWR?
+L power:GND #PWR0101
 U 1 1 5EA008E9
 P 2250 2400
-F 0 "#PWR?" H 2250 2150 50  0001 C CNN
+F 0 "#PWR0101" H 2250 2150 50  0001 C CNN
 F 1 "GND" H 2255 2227 50  0000 C CNN
 F 2 "" H 2250 2400 50  0001 C CNN
@@
 	2700 1600 2800 1600
 $Comp
-L Device:R R?
+L Device:R R1
 U 1 1 5EA0093D
 P 2800 1850
-F 0 "R?" H 2870 1896 50  0000 L CNN
+F 0 "R1" H 2870 1896 50  0000 L CNN
 F 1 "100k" H 2870 1805 50  0000 L CNN
-F 2 "" V 2730 1850 50  0001 C CNN
+F 2 "Resistor_THT:R_Axial_DIN0207_L6.3mm_D2.5mm_P7.62mm_Horizontal" V 2730 1850 50  0001 C CNN
 F 3 "~" H 2800 1850 50  0001 C CNN
 	1    2800 1850
@@
 	3100 2000 3100 1900
 $Comp
-L Switch:SW_SPDT SW?
+L Switch:SW_SPDT SW1
 U 1 1 5EA00F16
 P 3200 2200
-F 0 "SW?" V 3246 2012 50  0000 R CNN
+F 0 "SW1" V 3246 2012 50  0000 R CNN
 F 1 "SW_SPDT" V 3155 2012 50  0000 R CNN
-F 2 "" H 3200 2200 50  0001 C CNN
+F 2 "Connector_PinHeader_2.54mm:PinHeader_1x03_P2.54mm_Vertical" H 3200 2200 50  0001 C CNN
 F 3 "" H 3200 2200 50  0001 C CNN
 	1    3200 2200
@@
 Connection ~ 3100 2000
 $Comp
-L power:GND #PWR?
+L power:GND #PWR0102
 U 1 1 5EA00F9E
 P 4000 2400
-F 0 "#PWR?" H 4000 2150 50  0001 C CNN
+F 0 "#PWR0102" H 4000 2150 50  0001 C CNN
 F 1 "GND" H 4005 2227 50  0000 C CNN
 F 2 "" H 4000 2400 50  0001 C CNN
@@
 GND
 $Comp
-L power:PWR_FLAG #FLG?
+L power:PWR_FLAG #FLG0101
 U 1 1 5EA01067
 P 2500 2050
-F 0 "#FLG?" H 2500 2125 50  0001 C CNN
+F 0 "#FLG0101" H 2500 2125 50  0001 C CNN
 F 1 "PWR_FLAG" H 2500 2224 50  0000 C CNN
 F 2 "" H 2500 2050 50  0001 C CNN
@@
 Connection ~ 2250 2050
 $Comp
-L Regulator_Switching:R-783.3-0.5 U?
+L Regulator_Switching:R-783.3-0.5 U1
 U 1 1 5EA01405
 P 4000 1600
-F 0 "U?" H 4000 1842 50  0000 C CNN
+F 0 "U1" H 4000 1842 50  0000 C CNN
 F 1 "R-78E3.3-0.5" H 4000 1751 50  0000 C CNN
 F 2 "Converter_DCDC:Converter_DCDC_RECOM_R-78E-0.5_THT" H 4050 1350 50  0001 L CIN
@@
 	3500 1600 3700 1600
 $Comp
-L power:GND #PWR?
+L power:GND #PWR0103
 U 1 1 5EA01711
 P 3200 2400
-F 0 "#PWR?" H 3200 2150 50  0001 C CNN
+F 0 "#PWR0103" H 3200 2150 50  0001 C CNN
 F 1 "GND" H 3205 2227 50  0000 C CNN
 F 2 "" H 3200 2400 50  0001 C CNN
@@
 	4000 2400 4000 1900
 $Comp
-L Device:R R?
+L Device:R R2
 U 1 1 5EA01B14
 P 4500 1850
-F 0 "R?" H 4570 1896 50  0000 L CNN
+F 0 "R2" H 4570 1896 50  0000 L CNN
 F 1 "68" H 4570 1805 50  0000 L CNN
-F 2 "" V 4430 1850 50  0001 C CNN
+F 2 "Resistor_THT:R_Axial_DIN0207_L6.3mm_D2.5mm_P7.62mm_Horizontal" V 4430 1850 50  0001 C CNN
 F 3 "~" H 4500 1850 50  0001 C CNN
 	1    4500 1850
@@
 	4500 1600 4500 1700
 $Comp
-L Device:LED D?
+L Device:LED D1
 U 1 1 5EA01CA6
 P 4500 2150
-F 0 "D?" V 4538 2033 50  0000 R CNN
+F 0 "D1" V 4538 2033 50  0000 R CNN
 F 1 "LED(OSNG5113A)" V 4447 2033 50  0000 R CNN
-F 2 "" H 4500 2150 50  0001 C CNN
+F 2 "LED_THT:LED_D5.0mm" H 4500 2150 50  0001 C CNN
 F 3 "~" H 4500 2150 50  0001 C CNN
 	1    4500 2150
@@
 $EndComp
 $Comp
-L power:GND #PWR?
+L power:GND #PWR0104
 U 1 1 5EA01D1B
 P 4500 2400
-F 0 "#PWR?" H 4500 2150 50  0001 C CNN
+F 0 "#PWR0104" H 4500 2150 50  0001 C CNN
 F 1 "GND" H 4505 2227 50  0000 C CNN
 F 2 "" H 4500 2400 50  0001 C CNN
@@
 	4600 1600 4700 1600
 $Comp
-L Device:R R?
+L Device:R R3
 U 1 1 5EA02225
 P 4850 1600
-F 0 "R?" V 4643 1600 50  0000 C CNN
+F 0 "R3" V 4643 1600 50  0000 C CNN
 F 1 "10" V 4734 1600 50  0000 C CNN
-F 2 "" V 4780 1600 50  0001 C CNN
+F 2 "Resistor_THT:R_Axial_DIN0207_L6.3mm_D2.5mm_P7.62mm_Horizontal" V 4780 1600 50  0001 C CNN
 F 3 "~" H 4850 1600 50  0001 C CNN
 	1    4850 1600
@@
 $EndComp
 $Comp
-L Device:L L?
+L Device:L L1
 U 1 1 5EA022D4
 P 5250 1600
-F 0 "L?" V 5072 1600 50  0000 C CNN
+F 0 "L1" V 5072 1600 50  0000 C CNN
 F 1 "100u" V 5163 1600 50  0000 C CNN
-F 2 "" H 5250 1600 50  0001 C CNN
+F 2 "Inductor_THT:L_Axial_L7.0mm_D3.3mm_P10.16mm_Horizontal_Fastron_MICC" H 5250 1600 50  0001 C CNN
 F 3 "~" H 5250 1600 50  0001 C CNN
 	1    5250 1600
@@
 3.3VA
 $Comp
-L Device:C C?
+L Device:C C1
 U 1 1 5EA02A6C
 P 5500 1850
-F 0 "C?" H 5615 1896 50  0000 L CNN
+F 0 "C1" H 5615 1896 50  0000 L CNN
 F 1 "10u" H 5615 1805 50  0000 L CNN
-F 2 "" H 5538 1700 50  0001 C CNN
+F 2 "Capacitor_THT:C_Disc_D5.0mm_W2.5mm_P5.00mm" H 5538 1700 50  0001 C CNN
 F 3 "~" H 5500 1850 50  0001 C CNN
 	1    5500 1850
@@
 Connection ~ 5500 1600
 $Comp
-L Device:R R?
+L Device:R R4
 U 1 1 5EA02D76
 P 5900 1850
-F 0 "R?" H 5970 1896 50  0000 L CNN
+F 0 "R4" H 5970 1896 50  0000 L CNN
 F 1 "1k 1%" H 5970 1805 50  0000 L CNN
-F 2 "" V 5830 1850 50  0001 C CNN
+F 2 "Resistor_THT:R_Axial_DIN0207_L6.3mm_D2.5mm_P7.62mm_Horizontal" V 5830 1850 50  0001 C CNN
 F 3 "~" H 5900 1850 50  0001 C CNN
 	1    5900 1850
@@
 $EndComp
 $Comp
-L Device:R R?
+L Device:R R5
 U 1 1 5EA02DC6
 P 5900 2350
-F 0 "R?" H 5970 2396 50  0000 L CNN
+F 0 "R5" H 5970 2396 50  0000 L CNN
 F 1 "1k 1%" H 5970 2305 50  0000 L CNN
-F 2 "" V 5830 2350 50  0001 C CNN
+F 2 "Resistor_THT:R_Axial_DIN0207_L6.3mm_D2.5mm_P7.62mm_Horizontal" V 5830 2350 50  0001 C CNN
 F 3 "~" H 5900 2350 50  0001 C CNN
 	1    5900 2350
@@
 $EndComp
 $Comp
-L Device:C C?
+L Device:C C2
 U 1 1 5EA030B8
 P 6400 2350
-F 0 "C?" H 6515 2396 50  0000 L CNN
+F 0 "C2" H 6515 2396 50  0000 L CNN
 F 1 "0.1u" H 6515 2305 50  0000 L CNN
-F 2 "" H 6438 2200 50  0001 C CNN
+F 2 "Capacitor_THT:C_Disc_D5.0mm_W2.5mm_P5.00mm" H 6438 2200 50  0001 C CNN
 F 3 "~" H 6400 2350 50  0001 C CNN
 	1    6400 2350
@@
 	6400 2500 6400 2600
 $Comp
-L power:GND #PWR?
+L power:GND #PWR0105
 U 1 1 5EA04A64
 P 6400 2600
-F 0 "#PWR?" H 6400 2350 50  0001 C CNN
+F 0 "#PWR0105" H 6400 2350 50  0001 C CNN
 F 1 "GND" H 6405 2427 50  0000 C CNN
 F 2 "" H 6400 2600 50  0001 C CNN
@@
 $EndComp
 $Comp
-L power:GND #PWR?
+L power:GND #PWR0106
 U 1 1 5EA04A92
 P 5900 2600
-F 0 "#PWR?" H 5900 2350 50  0001 C CNN
+F 0 "#PWR0106" H 5900 2350 50  0001 C CNN
 F 1 "GND" H 5905 2427 50  0000 C CNN
 F 2 "" H 5900 2600 50  0001 C CNN
@@
 $EndComp
 $Comp
-L power:GND #PWR?
+L power:GND #PWR0107
 U 1 1 5EA04AB9
 P 5500 2600
-F 0 "#PWR?" H 5500 2350 50  0001 C CNN
+F 0 "#PWR0107" H 5500 2350 50  0001 C CNN
 F 1 "GND" H 5505 2427 50  0000 C CNN
 F 2 "" H 5500 2600 50  0001 C CNN
@@
 Text GLabel 6000 1600 2    50   Output ~ 0
 1.65V
+$Comp
+L power:PWR_FLAG #FLG0102
+U 1 1 5EA8392E
+P 3300 1250
+F 0 "#FLG0102" H 3300 1325 50  0001 C CNN
+F 1 "PWR_FLAG" H 3300 1424 50  0000 C CNN
+F 2 "" H 3300 1250 50  0001 C CNN
+F 3 "~" H 3300 1250 50  0001 C CNN
+	1    3300 1250
+	1    0    0    -1
+$EndComp
+Wire Wire Line
+	3300 1250 3500 1250
+Connection ~ 3500 1250
+$Comp
+L power:PWR_FLAG #FLG0104
+U 1 1 5EA85212
+P 5300 1250
+F 0 "#FLG0104" H 5300 1325 50  0001 C CNN
+F 1 "PWR_FLAG" H 5300 1424 50  0000 C CNN
+F 2 "" H 5300 1250 50  0001 C CNN
+F 3 "~" H 5300 1250 50  0001 C CNN
+	1    5300 1250
+	1    0    0    -1
+$EndComp
+Wire Wire Line
+	5300 1250 5500 1250
+Connection ~ 5500 1250
 $EndSCHEMATC
