File: PCB/_saved_Power.sch (KiCad schematic (older format))
At the start: 14 parts, among them J2 JST_XA_1x2, Q1 2SK4017, SW1 SW_SPDT, U1 R-78E3.3-0.5

Commit message: DXFを追加、部品配置を開始
Parts:
- F1: value RXEF160 -> MF-RX160; footprint (none) -> Cheese_Burger_Library:RF-RX160
- R1, R2, R3, R4, R5: footprint (none) -> Resistor_THT:R_Axial_DIN0207_L6.3mm_D2.5mm_P7.62mm_Horizontal
- SW1: footprint (none) -> Connector_PinHeader_2.54mm:PinHeader_1x03_P2.54mm_Vertical
Changed lines of the file:
@@
 P 2550 1600
 F 0 "F1" V 2325 1600 50  0000 C CNN
-F 1 "RXEF160" V 2416 1600 50  0000 C CNN
-F 2 "" H 2600 1400 50  0001 L CNN
+F 1 "MF-RX160" V 2416 1600 50  0000 C CNN
+F 2 "Cheese_Burger_Library:RF-RX160" H 2600 1400 50  0001 L CNN
 F 3 "~" H 2550 1600 50  0001 C CNN
 	1    2550 1600
@@
 F 0 "R1" H 2870 1896 50  0000 L CNN
 F 1 "100k" H 2870 1805 50  0000 L CNN
-F 2 "" V 2730 1850 50  0001 C CNN
+F 2 "Resistor_THT:R_Axial_DIN0207_L6.3mm_D2.5mm_P7.62mm_Horizontal" V 2730 1850 50  0001 C CNN
 F 3 "~" H 2800 1850 50  0001 C CNN
 	1    2800 1850
@@
 F 0 "SW1" V 3246 2012 50  0000 R CNN
 F 1 "SW_SPDT" V 3155 2012 50  0000 R CNN
-F 2 "" H 3200 2200 50  0001 C CNN
+F 2 "Connector_PinHeader_2.54mm:PinHeader_1x03_P2.54mm_Vertical" H 3200 2200 50  0001 C CNN
 F 3 "" H 3200 2200 50  0001 C CNN
 	1    3200 2200
@@
 F 0 "R2" H 4570 1896 50  0000 L CNN
 F 1 "68" H 4570 1805 50  0000 L CNN
-F 2 "" V 4430 1850 50  0001 C CNN
+F 2 "Resistor_THT:R_Axial_DIN0207_L6.3mm_D2.5mm_P7.62mm_Horizontal" V 4430 1850 50  0001 C CNN
 F 3 "~" H 4500 1850 50  0001 C CNN
 	1    4500 1850
@@
 F 0 "R3" V 4643 1600 50  0000 C CNN
 F 1 "10" V 4734 1600 50  0000 C CNN
-F 2 "" V 4780 1600 50  0001 C CNN
+F 2 "Resistor_THT:R_Axial_DIN0207_L6.3mm_D2.5mm_P7.62mm_Horizontal" V 4780 1600 50  0001 C CNN
 F 3 "~" H 4850 1600 50  0001 C CNN
 	1    4850 1600
@@
 F 0 "R4" H 5970 1896 50  0000 L CNN
 F 1 "1k 1%" H 5970 1805 50  0000 L CNN
-F 2 "" V 5830 1850 50  0001 C CNN
+F 2 "Resistor_THT:R_Axial_DIN0207_L6.3mm_D2.5mm_P7.62mm_Horizontal" V 5830 1850 50  0001 C CNN
 F 3 "~" H 5900 1850 50  0001 C CNN
 	1    5900 1850
@@
 F 0 "R5" H 5970 2396 50  0000 L CNN
 F 1 "1k 1%" H 5970 2305 50  0000 L CNN
-F 2 "" V 5830 2350 50  0001 C CNN
+F 2 "Resistor_THT:R_Axial_DIN0207_L6.3mm_D2.5mm_P7.62mm_Horizontal" V 5830 2350 50  0001 C CNN
 F 3 "~" H 5900 2350 50  0001 C CNN
 	1    5900 2350
@@
 	5900 1700 5900 1600
 Wire Wire Line
-	5900 1600 6000 1600
-Connection ~ 5900 1600
-Text GLabel 6000 1600 2    50   Output ~ 0
+	6400 2100 6500 2100
+Text GLabel 6500 2100 2    50   Output ~ 0
 1.65V
 $Comp
@@
 	5300 1250 5500 1250
 Connection ~ 5500 1250
+Connection ~ 6400 2100
 $EndSCHEMATC
